Commit message: Added camera to robot model

File: ros_ws/src/intro_robot_description/urdf/four_wheel_bot.xacro (robot description, xacro)
@@ -8,4 +8,8 @@
     <xacro:property name="length" value="1.4" />    <!-- Y dimension -->
     <xacro:property name="depth" value="0.5" />    <!-- Z dimension -->
+    <xacro:property name="camera_len" value="0.125" /> <!-- Camera square side length -->
+    <!-- ==== Include files ==== -->
+    <!-- Gazebo file include -->
+    <xacro:include filename="four_wheel_bot.gazebo" />
     <!-- ==== Macros ==== -->
     <!-- Attach the wheel at Pitch -1.57079632679 -->
@@ -48,5 +52,6 @@
     </xacro:macro>
     <!-- ==== Main code ==== -->
-    <!-- Links -->
+    <!-- === Links === -->
+    <!-- Base link -->
     <link name="base_link">
         <collision>
@@ -81,5 +86,32 @@
     <!-- Back left wheel -->
     <xacro:attach_wheels name="bl" x="${-width/2}" y="${-length/2}" reflect="1" />
-    <!-- Gazebo file include -->
-    <xacro:include filename="four_wheel_bot.gazebo" />
+    <!-- Camera sensor joint -->
+    <joint name="joint_name" type="fixed">
+        <parent link="base_link" />
+        <child link="camera_link" />
+        <origin xyz="0.0 ${length/2 - camera_len/2} ${depth}" rpy="0.0 0.0 1.57079632679" />
+    </joint>
+    <!-- Camera sensor link -->
+    <link name="camera_link">
+        <collision>
+            <origin xyz="0.0 0.0 ${camera_len/2}"/>
+            <geometry>
+                <box size="${camera_len} ${camera_len} ${camera_len}"/>
+            </geometry>
+        </collision>
+        <visual>
+            <origin xyz="0.0 0.0 ${camera_len/2}"/>
+            <geometry>
+                <box size="${camera_len} ${camera_len} ${camera_len}"/>
+            </geometry>
+            <material name="red" />
+        </visual>
+        <inertial>
+            <origin xyz="0.0 0.0 0.0" rpy="0.0 0.0 0.0"/>
+            <mass value="0.1"/>
+            <inertia ixx="1.0" ixy="0.0" ixz="0.0"
+                               iyy="1.0" iyz="0.0"
+                                         izz="1.0"/>
+        </inertial>
+    </link>
 </robot>
